File: pcb/dmx-eth-dimmer.kicad_pcb (KiCad board)
At the start: 2 copper layers, 200.7 x 123.2 mm, 114 parts, among them J1 MAINS IN, J10 LOAD, J11 CH4 PRG, J12 LOAD, J13 CH6 PRG, J14 LOAD, J15 CH7 PRG, J16 LOAD, J17 PRG, J18 LOAD, J19 CH8 PRG, J2 STANDARD ENC28J60, J20 LOAD, J3 MINI ENC28J60, J4 MASTER PROG, J5 CH1 PRG, J6 LOAD, J7 CH2 PRG, J8 LOAD, J9 CH5 PRG, SW1 IP1, SW2 IP2, SW3 IP3, SW4 IP4, SW5 DMXAH, SW6 DMXAL, SW7 SW_DIP_x08, U1 PSU-5VDC, U10 MOC3020M, U11 PIC12(L)F1571/2, U12 MOC3020M, U13 PIC12(L)F1571/2, U14 MOC3020M, U15 PIC12(L)F1571/2, U16 MOC3020M, U17 PIC12(L)F1571/2, U18 MOC3020M, U19 PIC12(L)F1571/2, U2 3.3v Regulator, U20 MOC3020M, U3 74HCT08, U4 4N25, U5 PIC12(L)F1571/2, U6 MOC3020M, U7 PIC12(L)F1571/2, U8 MOC3020M, U9 PIC12(L)F1571/2, Y1 20MHz

Commit message: Updated PCB
Parts:
- moved R26 2.01 mm to (171.4, 101.0)
- moved R12 1.91 mm to (159.4, 113.0)
Routing:
- net GND: track 796.5 -> 854.6 mm
- net Net-(R26-Pad2): track 11.3 -> 6.92 mm
- net Net-(J5-Pad5): track 25.2 -> 27.1 mm
- net ZC: track 335.6 -> 337.5 mm
- net Net-(J19-Pad5): track 17.5 -> 18.9 mm
- net Net-(R12-Pad2): track 8.19 -> 7.03 mm
- net 5V: track 645.6 -> 646.7 mm

Commit message: PWM1/TMR1 version
Parts:
- added R30: 10K, Resistors_THT:R_Axial_DIN0207_L6.3mm_D2.5mm_P10.16mm_Horizontal, F.Cu at (58.4, 82.5)
- D1: value CFG -> CFG Status
- D2: value ETH -> Ethernet Status
- J11: value CH4 PRG -> PRG
- J13: value CH6 PRG -> PRG
- J15: value CH7 PRG -> PRG
- J19: value CH8 PRG -> PRG
- J5: value CH1 PRG -> PRG
- J7: value CH2 PRG -> PRG
- J9: value CH5 PRG -> PRG
- moved J7 1.27 mm to (103.5, 106.7)
Connections:
- U11 pad 3: CHNCLK -> ZC
- U11 pad 5: ZC -> CHNCLK
- U13 pad 3: CHNCLK -> ZC
- U13 pad 5: ZC -> CHNCLK
- U15 pad 3: CHNCLK -> ZC
- U15 pad 5: ZC -> CHNCLK
- U17 pad 3: CHNCLK -> ZC
- U17 pad 5: ZC -> CHNCLK
- U19 pad 3: CHNCLK -> ZC
- U19 pad 5: ZC -> CHNCLK
- U5 pad 3: CHNCLK -> ZC
- U5 pad 5: ZC -> CHNCLK
- U7 pad 3: CHNCLK -> ZC
- U7 pad 5: ZC -> CHNCLK
- U9 pad 3: CHNCLK -> ZC
- U9 pad 5: ZC -> CHNCLK
Routing:
- net CHNCLK: track 311.4 -> 352.9 mm, vias 10 -> 12
- net ZC: track 337.5 -> 329.2 mm, vias 12 -> 14
- net /MCLR: track 24.9 -> 30.0 mm
- net 5V: track 646.7 -> 649.8 mm
- net Net-(J7-Pad5): track 15.6 -> 18.1 mm
- net /CH2: track 47.9 -> 49.8 mm
- net GND: track 854.6 -> 856.2 mm
- net Net-(J7-Pad1): track 5.08 -> 6.35 mm
